Commit message: 传感器仿真结束 2025/9/13

File: chapt6/chapt6_ws/install/zzs_description/share/zzs_description/urdf/plugins/gazebo_control_plugin.xacro (robot description, xacro)
@@ -2,31 +2,29 @@
 <robot xmlns:xacro="http://www.ros.org/wiki/xacro">
     <xacro:macro name="gazebo_control_plugin">
-        <!-- 差速驱动 + odom + tf -->
         <gazebo>
-            <plugin filename="gz-sim-diff-drive-system" name="gz::sim::systems::DiffDrive">
+            <plugin name='diff_drive' filename='libgazebo_ros_diff_drive.so'>
+                <ros>
+                    <namespace>/</namespace>
+                    <remapping>cmd_vel:=cmd_vel</remapping>
+                    <remapping>odom:=odom</remapping>
+                </ros>
+                <update_rate>30</update_rate>
+                <!-- wheels -->
                 <left_joint>left_wheel_joint</left_joint>
                 <right_joint>right_wheel_joint</right_joint>
+                <!-- kinematics -->
                 <wheel_separation>0.2</wheel_separation>
-                <wheel_radius>0.032</wheel_radius>
-                <topic>cmd_vel</topic>
-                <odom_topic>odom</odom_topic>
-                <odom_publish_frequency>30</odom_publish_frequency>
-                <!-- ★★★ 关键修改：显式指定 TF 话题与 frame ★★★ -->
-                <tf_topic>/tf</tf_topic>
-                <frame_id>odom</frame_id>
-                <child_frame_id>base_footprint</child_frame_id>
-                <max_linear_acceleration>1.0</max_linear_acceleration>
-                <max_angular_acceleration>1.0</max_angular_acceleration>
+                <wheel_diameter>0.064</wheel_diameter>
+                <!-- limits -->
+                <max_wheel_torque>20</max_wheel_torque>
+                <max_wheel_acceleration>1.0</max_wheel_acceleration>
+                <!-- output -->
+                <publish_odom>true</publish_odom>
+                <publish_odom_tf>true</publish_odom_tf>
+                <publish_wheel_tf>true</publish_wheel_tf>
+                <odometry_frame>odom</odometry_frame>
+                <robot_base_frame>base_footprint</robot_base_frame>
             </plugin>
         </gazebo>
-        <!-- 关节状态（保持不变） -->
-        <gazebo>
-            <plugin filename="gz-sim-joint-state-publisher-system" name="gz::sim::systems::JointStatePublisher">
-                <topic>joint_states</topic>
-                <joint_name>left_wheel_joint</joint_name>
-                <joint_name>right_wheel_joint</joint_name>
-                <update_rate>30</update_rate>
-            </plugin>
-        </gazebo>
-    </xacro:macro>
+   </xacro:macro>
 </robot>

File: chapt6/chapt6_ws/install/zzs_description/share/zzs_description/urdf/plugins/gazebo_sensor_plugin.xacro (robot description, xacro)
@@ -2,26 +2,36 @@
 <robot xmlns:xacro="http://www.ros.org/wiki/xacro">
     <xacro:macro name="gazebo_sensor_plugin">
-        <!-- 激光雷达传感器，2D 单线 -->
-        <!-- ★ reference 改为 base_footprint（融合后的实际 link） -->
-        <gazebo reference="base_footprint">
-            <sensor name="laser" type="gpu_lidar">
-                <topic>/scan</topic>
-                <update_rate>10</update_rate>
+                <gazebo reference="laser_link">
+            <sensor name="laserscan" type="ray">
+                <plugin name="laserscan" filename="libgazebo_ros_ray_sensor.so">
+                    <ros>
+                        <namespace>/</namespace>
+                        <remapping>~/out:=scan</remapping>
+                    </ros>
+                    <output_type>sensor_msgs/LaserScan</output_type>
+                    <frame_name>laser_link</frame_name>
+                </plugin>
                 <always_on>true</always_on>
                 <visualize>true</visualize>
-                <lidar>
+                <update_rate>5</update_rate>
+                <pose>0 0 0 0 0 0</pose>
+								<!-- 激光传感器配置 -->
+                <ray>
+                    <!-- 设置扫描范围 -->
                     <scan>
                         <horizontal>
                             <samples>360</samples>
-                            <resolution>1</resolution>
-                            <min_angle>-3.14159</min_angle>
-                            <max_angle>3.14159</max_angle>
+                            <resolution>1.000000</resolution>
+                            <min_angle>0.000000</min_angle>
+                            <max_angle>6.280000</max_angle>
                         </horizontal>
                     </scan>
+                    <!-- 设置扫描距离 -->
                     <range>
-                        <min>0.12</min>
-                        <max>12.0</max>
-                        <resolution>0.01</resolution>
+                        <min>0.120000</min>
+                        <max>8.0</max>
+                        <resolution>0.015000</resolution>
                     </range>
+                    <!-- 设置噪声 -->
                     <noise>
                         <type>gaussian</type>
@@ -29,5 +39,98 @@
                         <stddev>0.01</stddev>
                     </noise>
-                </lidar>
+                </ray>
+            </sensor>
+        </gazebo>
+        <gazebo reference="imu_link">
+            <sensor name="imu_sensor" type="imu">
+                <plugin name="imu_plugin" filename="libgazebo_ros_imu_sensor.so">
+                    <ros>
+                        <namespace>/</namespace>
+                        <remapping>~/out:=imu</remapping>
+                    </ros>
+                    <initial_orientation_as_reference>false</initial_orientation_as_reference>
+                </plugin>
+                <update_rate>100</update_rate>
+                <always_on>true</always_on>
+                <!-- 六轴噪声设置 -->
+                <imu>
+                    <angular_velocity>
+                        <x>
+                            <noise type="gaussian">
+                                <mean>0.0</mean>
+                                <stddev>2e-4</stddev>
+                                <bias_mean>0.0000075</bias_mean>
+                                <bias_stddev>0.0000008</bias_stddev>
+                            </noise>
+                        </x>
+                        <y>
+                            <noise type="gaussian">
+                                <mean>0.0</mean>
+                                <stddev>2e-4</stddev>
+                                <bias_mean>0.0000075</bias_mean>
+                                <bias_stddev>0.0000008</bias_stddev>
+                            </noise>
+                        </y>
+                        <z>
+                            <noise type="gaussian">
+                                <mean>0.0</mean>
+                                <stddev>2e-4</stddev>
+                                <bias_mean>0.0000075</bias_mean>
+                                <bias_stddev>0.0000008</bias_stddev>
+                            </noise>
+                        </z>
+                    </angular_velocity>
+                    <linear_acceleration>
+                        <x>
+                            <noise type="gaussian">
+                                <mean>0.0</mean>
+                                <stddev>1.7e-2</stddev>
+                                <bias_mean>0.1</bias_mean>
+                                <bias_stddev>0.001</bias_stddev>
+                            </noise>
+                        </x>
+                        <y>
+                            <noise type="gaussian">
+                                <mean>0.0</mean>
+                                <stddev>1.7e-2</stddev>
+                                <bias_mean>0.1</bias_mean>
+                                <bias_stddev>0.001</bias_stddev>
+                            </noise>
+                        </y>
+                        <z>
+                            <noise type="gaussian">
+                                <mean>0.0</mean>
+                                <stddev>1.7e-2</stddev>
+                                <bias_mean>0.1</bias_mean>
+                                <bias_stddev>0.001</bias_stddev>
+                            </noise>
+                        </z>
+                    </linear_acceleration>
+                </imu>
+            </sensor>
+        </gazebo>
+        <gazebo reference="camera_link">
+            <sensor type="depth" name="camera_sensor">
+                <plugin name="depth_camera" filename="libgazebo_ros_camera.so">
+                    <frame_name>camera_optical_link</frame_name>
+                </plugin>
+                <always_on>true</always_on>
+                <update_rate>10</update_rate>
+                <camera name="camera">
+                    <horizontal_fov>1.5009831567</horizontal_fov>
+                    <image>
+                        <width>800</width>
+                        <height>600</height>
+                        <format>R8G8B8</format>
+                    </image>
+                    <distortion>
+                        <k1>0.0</k1>
+                        <k2>0.0</k2>
+                        <k3>0.0</k3>
+                        <p1>0.0</p1>
+                        <p2>0.0</p2>
+                        <center>0.5 0.5</center>
+                    </distortion>
+                </camera>
             </sensor>
         </gazebo>

File: chapt6/chapt6_ws/install/zzs_description/share/zzs_description/urdf/sensor/camera.urdf.xacro (robot description, xacro)
@@ -17,4 +17,5 @@
                 <xacro:box_inertia m="0.1" w="0.02" h="0.10" d="0.02"/>
             </link>
+            <link name="camera_optical_link"></link>
         <joint name="camera_joint" type="fixed">
             <origin xyz="${xyz}" rpy="0.0 0.0 0.0"/>
@@ -22,4 +23,9 @@
             <child link="camera_link"/>
         </joint>
+        <joint name="camera_optical_joint" type="fixed">
+            <origin xyz="0 0 0" rpy="${pi/2} 0.0 ${pi/2}"/>
+            <parent link="camera_link"/>
+            <child link="camera_optical_link"/>
+        </joint>
     </xacro:macro>
 </robot>
